File: numpad.sch (KiCad schematic (older format))
At the start: 54 parts, among them J2 Conn_01x06, SW1 RESET, SW2 BOOT

Commit message: fix mistakes
Parts:
- removed D14: D_Small, Diode_THT:D_DO-35_SOD27_P7.62mm_Horizontal, symbol Device:D_Small
- removed J2: Conn_01x06, Connector_PinHeader_2.54mm:PinHeader_1x06_P2.54mm_Vertical, symbol Connector_Generic:Conn_01x06
- removed MX12: MX-NoLED, MX_Only:MXOnly-1U-NoLED, symbol MX_Alps_Hybrid:MX-NoLED
- added D17, D21, D22, D23: D_Small, Diode_THT:D_DO-35_SOD27_P7.62mm_Horizontal, symbol Device:D_Small
- added ISP1: AVR-ISP-6, Connector_PinHeader_2.54mm:PinHeader_2x03_P2.54mm_Horizontal, symbol Connector:AVR-ISP-6
- added MX15, MX19, MX21: MX-NoLED, MX_Only:MXOnly-2U-NoLED, symbol MX_Alps_Hybrid:MX-NoLED
- added MX20: MX-NoLED, MX_Only:MXOnly-1U-NoLED, symbol MX_Alps_Hybrid:MX-NoLED
- D1, D2: value D_Zener -> 3.6V
- MCU1: footprint Package_DIP:DIP-28_W7.62mm_Socket -> Package_DIP:DIP-28_W7.62mm
- MX16, MX18: footprint MX_Only:MXOnly-2U-NoLED -> MX_Only:MXOnly-1U-NoLED
- renumbered D15 to D14, D16 to D15, D17 to D16, MX13 to MX12, MX14 to MX13, MX15 to MX14
Connections:
- net +5V: now also ISP1.2 (VCC)
- net GND: now also ISP1.6 (GND)
- net MISO: now also ISP1.1 (MISO)
- net MOSI: now also ISP1.4 (MOSI)
- net SCK: now also ISP1.3 (SCK)
- net col0: now also MX19.2 (ROW)
- net col1: now also MCU1.13 (PD7), MX17.2 (ROW); no longer MCU1.15 (PB1)
- net col2: now also MCU1.15 (PB1), MX18.2 (ROW), MX20.2 (ROW); no longer MCU1.16 (PB2), MX17.2 (ROW)
- net col3: now also MCU1.16 (PB2), MX15.2 (ROW), MX21.2 (ROW); no longer MCU1.23 (PC0), MX18.2 (ROW)
- net reset: now also ISP1.5 (~RST)
- net row3: now also D17.1 (K)
- new net: D17.2 (A), MX15.1 (COL)
- new net: D21.2 (A), MX19.1 (COL)
- new net: D22.2 (A), MX20.1 (COL)
- new net: D23.2 (A), MX21.1 (COL)
- new net row5: D21.1 (K), D22.1 (K), D23.1 (K), MCU1.23 (PC0)
Other:
- moved on the sheet: D10, D11, D12, D13, D14, D15, D16, D18, D19, D20, D3, D4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

Commit message: update
Parts:
- removed USB1: USB_B_Mini, custom_parts:USB_Mini, symbol Connector:USB_B_Mini
- added R4, R5: 5.1K, Resistor_THT:R_Axial_DIN0204_L3.6mm_D1.6mm_P7.62mm_Horizontal, symbol Device:R
- added USB1: USB_C_Receptacle_USB2.0, custom_parts:USB_C_GCT_USB4085, symbol Connector:USB_C_Receptacle_USB2.0
- renumbered R4 to R6
Connections:
- net D+: now also R2.1; no longer R1.1
- net D-: now also R1.1; no longer R2.1
- net GND: now also R4.1, R5.1, USB1.A1 (GND), USB1.A12 (GND), USB1.B1 (GND), USB1.B12 (GND), USB1.S1 (SHIELD)
- net VCC: now also USB1.A4 (VBUS), USB1.A9 (VBUS), USB1.B4 (VBUS), USB1.B9 (VBUS)
- net col0: now also MCU1.23 (PC0); no longer MCU1.14 (PB0)
- net col1: now also MCU1.24 (PC1); no longer MCU1.13 (PD7)
- net col2: now also MCU1.25 (PC2); no longer MCU1.15 (PB1)
- net col3: now also MCU1.26 (PC3); no longer MCU1.16 (PB2)
- net row2: now also MCU1.16 (PB2); no longer MCU1.26 (PC3)
- net row3: now also MCU1.15 (PB1); no longer MCU1.25 (PC2)
- net row4: now also MCU1.13 (PD7); no longer MCU1.24 (PC1)
- net row5: now also MCU1.14 (PB0); no longer MCU1.23 (PC0)
- net at D2.1 (K), R2.2: now also USB1.A6 (D+), USB1.B6 (D+); no longer R3.1
- net at D1.1 (K), R1.2: now also R3.1, USB1.A7 (D-), USB1.B7 (D-)
- new net: R4.2, USB1.A5 (CC1)
- new net: R5.2, USB1.B5 (CC2)
Other:
- moved on the sheet: D1, D2, F1, ISP1, R1, R2, R3
