File: numpad.kicad_pcb (KiCad board)
At the start: 2 copper layers, 99.3 x 96.5 mm, 54 parts, among them J2 Conn_01x06, SW1 RESET, SW2 BOOT

Commit message: fix mistakes
Parts:
- removed the D14 at (159.0, 94.2)
- removed J2: Conn_01x06, Connector_PinHeader_2.54mm:PinHeader_1x06_P2.54mm_Vertical
- removed the MX12 at (168.5, 90.7)
- added D17: D_Small, Diode_THT:D_DO-35_SOD27_P7.62mm_Horizontal, F.Cu at (159.0, 107.7)
- added D21: D_Small, Diode_THT:D_DO-35_SOD27_P7.62mm_Horizontal, F.Cu at (101.9, 137.7)
- added D22: D_Small, Diode_THT:D_DO-35_SOD27_P7.62mm_Horizontal, F.Cu at (140.0, 137.8)
- added D23: D_Small, Diode_THT:D_DO-35_SOD27_P7.62mm_Horizontal, F.Cu at (159.0, 137.8)
- added G***: LOGO, custom_parts:elmo, B.Cu at (146.8, 80.3)
- added G***: LOGO, custom_parts:oshw, B.Cu at (123.4, 80.5)
- added ISP1: AVR-ISP-6, Connector_PinHeader_2.54mm:PinHeader_2x03_P2.54mm_Horizontal, F.Cu at (92.2, 139.4)
- added MX15: MX-NoLED, MX_Only:MXOnly-2U-NoLED, F.Cu at (168.5, 100.2)
- added MX19: MX-NoLED, MX_Only:MXOnly-2U-NoLED, F.Cu at (120.9, 147.8)
- added MX20: MX-NoLED, MX_Only:MXOnly-1U-NoLED, F.Cu at (149.5, 147.8)
- added MX21: MX-NoLED, MX_Only:MXOnly-2U-NoLED, F.Cu at (168.5, 138.3)
- D1, D2: value D_Zener -> 3.6V
- MCU1: footprint Package_DIP:DIP-28_W7.62mm_Socket -> Package_DIP:DIP-28_W7.62mm
- MX16, MX18: footprint MX_Only:MXOnly-2U-NoLED -> MX_Only:MXOnly-1U-NoLED
- moved SW2 22.2 mm to (93.2, 151.0)
- moved SW1 21.7 mm to (83.3, 151.0)
- moved MX18 21.3 mm to (149.5, 128.8), turned to 0 degrees
- moved R4 19.6 mm to (87.6, 147.8)
- moved D20 19.3 mm to (140.0, 118.9)
- moved D19 19.1 mm to (120.9, 118.9)
- moved MX17 19.1 mm to (130.4, 128.8)
- moved MX16 9.52 mm to (111.4, 128.8)
- moved C3 0.25 mm to (97.5, 94.7)
- renumbered D15 to D14, D16 to D15, D17 to D16, MX13 to MX12, MX14 to MX13, MX15 to MX14
Connections:
- MCU1 pad 13: Net-(MCU1-Pad13) -> col1
- MCU1 pad 15: col1 -> col2
- MCU1 pad 16: col2 -> col3
- MCU1 pad 23: col3 -> row5
- MX17 pad 2: col2 -> col1
- MX18 pad 2: col3 -> col2
Routing:
- net row5: track 0.00 -> 110.0 mm
- net col1: track 101.7 -> 139.3 mm
- net col2: track 138.0 -> 166.5 mm
- net col0: track 116.0 -> 142.2 mm
- net +5V: track 106.7 -> 129.7 mm
- net row3: track 71.7 -> 94.4 mm
- net reset: track 73.4 -> 95.5 mm
- net boot: track 57.1 -> 79.0 mm
- net row4: track 94.9 -> 74.8 mm
- net MOSI: track 21.8 -> 41.8 mm
- net row2: track 74.2 -> 55.2 mm
- net SCK: track 30.0 -> 47.4 mm
- net col3: track 154.0 -> 169.6 mm
- net Net-(D21-Pad2): track 0.00 -> 15.2 mm
- net MISO: track 26.1 -> 40.7 mm
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Other:
- board size 99.3 x 96.5 mm -> 99.3 x 115.8 mm
- board text added: "ELMOPAD"
- board text added: "rev1"

Commit message: ISP routing improvements
Routing:
- net MOSI: track 41.8 -> 38.8 mm
- net GND: track 8.77 -> 11.6 mm
- net boot: track 79.0 -> 79.6 mm

Commit message: add giant elmo logo
Parts:
- added G***: LOGO, custom_parts:elmo_big, B.Cu at (145.8, 100.1)
- G*** (x2): moved to F.Cu
- moved G*** 24.4 mm to (147.8, 81.0), turned to 0 degrees
- moved G*** 22.4 mm to (124.5, 80.8), turned to 0 degrees

Commit message: update
Parts:
- removed the G*** at (145.8, 100.1)
- added R4: 5.1K, Resistor_THT:R_Axial_DIN0204_L3.6mm_D1.6mm_P7.62mm_Horizontal, F.Cu at (98.2, 62.5)
- added R5: 5.1K, Resistor_THT:R_Axial_DIN0204_L3.6mm_D1.6mm_P7.62mm_Horizontal, F.Cu at (95.4, 62.5)
- added REF**: screw_hole, custom_parts:screw_hole, F.Cu at (91.2, 61.7)
- added REF**: screw_hole, custom_parts:screw_hole, F.Cu at (91.2, 146.8)
- added REF**: screw_hole, custom_parts:screw_hole, F.Cu at (101.9, 133.3)
- added REF**: screw_hole, custom_parts:screw_hole, F.Cu at (159.0, 133.3)
- added REF**: screw_hole, custom_parts:screw_hole, F.Cu at (101.9, 62.1)
- added REF**: screw_hole, custom_parts:screw_hole, F.Cu at (159.0, 62.1)
- G*** (x2): moved to B.Cu
- USB1: value USB_B_Mini -> USB_C_Receptacle_USB2.0; footprint custom_parts:USB_Mini -> custom_parts:USB_C_GCT_USB4085
- moved G*** 31.0 mm to (123.1, 99.7), turned to 180 degrees
- moved G*** 28.8 mm to (146.4, 99.4), turned to 180 degrees
- moved R6 19.6 mm to (87.9, 128.3)
- moved ISP1 3.05 mm to (95.2, 139.4)
- moved C1 2.84 mm to (90.2, 56.4)
- moved D21 2.79 mm to (101.9, 140.5)
- moved F1 1.05 mm to (85.6, 61.0)
- moved USB1 0.13 mm to (91.1, 43.2), turned to 180 degrees
- renumbered SW2 to BOOT, R4 to R6, SW1 to RESET
Connections:
- MCU1 pad 13: col1 -> row4
- MCU1 pad 14: col0 -> row5
- MCU1 pad 15: col2 -> row3
- MCU1 pad 16: col3 -> row2
- MCU1 pad 23: row5 -> col0
- MCU1 pad 24: row4 -> col1
- MCU1 pad 25: row3 -> col2
- MCU1 pad 26: row2 -> col3
- R1 pad 1: D+ -> D-
- R2 pad 1: D- -> D+
- R3 pad 1: Net-(D2-Pad1) -> Net-(D1-Pad1)
Routing:
- net GND: track 11.6 -> 117.0 mm, vias 0 -> 1
- net row3: track 94.4 -> 69.3 mm
- net Net-(R5-Pad2): track 0.00 -> 21.2 mm
- net Net-(D1-Pad1): track 33.3 -> 53.4 mm, vias 0 -> 1
- net col1: track 139.3 -> 122.0 mm
- net row4: track 74.8 -> 58.5 mm
- net col0: track 142.2 -> 127.8 mm
- net Net-(D2-Pad1): track 33.2 -> 45.9 mm, vias 0 -> 1
- net col3: track 169.6 -> 181.1 mm
- net Net-(R4-Pad2): track 0.00 -> 9.48 mm
- net VCC: track 6.87 -> 16.2 mm
- net +5V: track 129.7 -> 138.1 mm
- net col2: track 166.5 -> 158.6 mm
- net row5: track 110.0 -> 105.2 mm
- net reset: track 95.5 -> 100.0 mm
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Other:
- board text added: "rev2"
- board text removed: "rev1"

Commit message: update
Parts:
- moved G*** 20.0 mm to (147.8, 79.5)
- moved G*** 20.0 mm to (124.5, 79.8)
Other:
- board text added: "github.com/kb-elmo/numpad elmo.space"
